Commit message: ur3_planning & ur_modern_driver

File: ur_description/urdf/ur3.urdf.xacro (robot description, xacro)
@@ -289,4 +289,7 @@
       <parent link="${prefix}wrist_3_link"/>
       <child link="${prefix}tool0"/>
+      <!-- <geometry>
+         <mesh filename="package://ur_description/meshes/ur3/collision/pg70.dae"/>
+      </geometry> -->
     </joint>
   </xacro:macro>
