Commit message: ur3_pg70

File: ur_description/urdf/ur3_pg70_table.urdf.xacro (robot description, xacro)
@@ -1,5 +1,5 @@
 <?xml version="1.0"?>
 <robot xmlns:xacro="http://ros.org/wiki/xacro"
-       name="ur3_pg70" >
+       name="ur3_pg70_table" >
   <!-- common stuff -->
   <xacro:include filename="$(find ur_description)/urdf/common.gazebo.xacro" />
@@ -11,9 +11,24 @@
   <xacro:ur3_robot prefix="" joint_limited="false"/>
   <link name="world" />
+<!-- box-->
+  <link name="box_link">
+    <visual>
+      <geometry>
+        <box size="1.0 1.0 0.86"/>
+      </geometry>
+    </visual>
+  </link>
+<!-- attach the box to the world-->
   <joint name="world_joint" type="fixed">
     <parent link="world" />
-    <child link = "base_link" />
-    <origin xyz="0.0 0.0 0.0" rpy="0.0 0.0 0.0" />
+    <child link = "box_link" />
+    <origin xyz="0.0 0.0 0.43" rpy="0.0 0.0 0.0" />
   </joint>
+<!-- attach the robot to the box -->
+ <joint name="box_joint" type="fixed">
+    <parent link="box_link"/>
+    <child link="base_link"/>
+    <origin xyz="0.0 0.0 0.43" rpy="0 0 1.57" />
+ </joint>
  <link name="gripper_link">
     <visual>

File: ur_description/urdf/ur3_table.urdf.xacro (robot description, xacro)
@@ -4,5 +4,5 @@
   <!-- common stuff -->
   <xacro:include filename="$(find ur_description)/urdf/common.gazebo.xacro" />
-  <!-- ur5 -->
+  <!-- ur3 -->
   <xacro:include filename="$(find ur_description)/urdf/ur3.urdf.xacro" />
   <!-- arm -->
@@ -29,9 +29,3 @@
     <origin xyz="0.0 0.0 0.43" rpy="0 0 1.57" />
  </joint>
-  <!-- GRIPPER -->
-  <!-- Import robotiq gazebo and gripper description -->
-  <!--xacro:include filename="$(find robotiq_85_description)/urdf/robotiq_85_gripper.urdf.xacro" />
-  <xacro:robotiq_85_gripper prefix="" parent="ee_link" >
-        <origin xyz="0 0 0" rpy="0 0 0"/>
-    </xacro:robotiq_85_gripper-->
 </robot>
