Commit message: ur3_pg70_running

File: ur_description/urdf/ur3_pg70_old.urdf.xacro (robot description, xacro)
@@ -9,17 +9,39 @@
   <xacro:ur3_robot prefix="" joint_limited="false"/>
   <link name="world" />
+  <link name="box_link">
+    <visual>
+      <geometry>
+        <box size="1.0 1.0 0.86"/>
+      </geometry>
+    </visual>
+    <inertial>
+        <origin xyz="0 0 0" rpy="0 0 0"/>
+        <mass value="100"/>
+        <inertia ixx="1.0" ixy="0" ixz="0" iyy="1.0" iyz="0" izz="1.0" />
+    </inertial>
+    <collision>
+      <geometry>
+        <box size="1.0 1.0 0.86"/>
+      </geometry>
+    </collision>
+  </link>
   <joint name="world_joint" type="fixed">
     <parent link="world" />
-    <child link = "base_link" />
-    <origin xyz="0.0 0.0 0.0" rpy="0.0 0.0 0.0" />
+    <child link = "box_link" />
+    <origin xyz="0.0 0.0 0.43" rpy="0.0 0.0 0.0" />
   </joint>
+   <joint name="box_joint" type="fixed">
+    <parent link="box_link"/>
+    <child link="base_link"/>
+    <origin xyz="0.0 0.0 0.43" rpy="0 0 1.57" />
+ </joint>
  <link name="gripper_link">
     <visual>
       <geometry>
         <box size="0.08 0.113 0.005"/>
-         <material name="o">
-          <color rgba="0.549019608 0.450980392 0.235294118 1" />
-         </material>
       </geometry>
+      <material name="o">
+        <color rgba="0.549019608 0.450980392 0.235294118 1" />
+      </material>
     </visual>
     <inertial>
@@ -28,4 +50,9 @@
         <inertia ixx="0.0001" ixy="0" ixz="0" iyy="0.0001" iyz="0" izz="0.0001" />
     </inertial>
+    <collision>
+      <geometry>
+        <box size="0.08 0.113 0.005"/>
+      </geometry>
+    </collision>
   </link>
   <joint name="gripper_joint" type="fixed">
@@ -52,4 +79,9 @@
         <inertia ixx="0.0001" ixy="0" ixz="0" iyy="0.0001" iyz="0" izz="0.0001" />
     </inertial>
+    <collision>
+      <geometry>
+        <cylinder length="0.03" radius="0.0075"/>
+      </geometry>
+    </collision>
  </link>
  <joint name="gripper_power_cable_joint" type="fixed">
@@ -93,8 +125,8 @@
  </joint>-->
   <gazebo>
-      <plugin name="ros_control" filename="libgazebo_ros_control.so">
-        <!--robotNamespace>/</robotNamespace-->
-        <!--robotSimType>gazebo_ros_control/DefaultRobotHWSim</robotSimType-->
+      <plugin name="gazebo_ros_control" filename="libgazebo_ros_control.so">
+        <!--<robotNamespace>ur3_pg70</robotNamespace>-->
+         <robotSimType>gazebo_ros_control/DefaultRobotHWSim</robotSimType>
       </plugin>
-    </gazebo>
+  </gazebo>
 </robot>
