Commit message: ur3_pg70_controller

File: ur_description/urdf/ur3_pg70.urdf.xacro (robot description, xacro)
@@ -7,5 +7,5 @@
   <xacro:include filename="$(find ur_description)/urdf/ur3.urdf.xacro" />
   <!-- schunk pg70 -->
-  <xacro:include filename="$(find schunk_pg70)/urdf/pg70.urdf.xacro" />
+  <xacro:include filename="$(find schunkPG70_description)/robots/schunkPG70_description.URDF" />
   <!-- arm -->
   <xacro:ur3_robot prefix="" joint_limited="false"/>
@@ -21,4 +21,7 @@
         <box size="0.08 0.113 0.005"/>
       </geometry>
+      <material name="o">
+      	 <color rgba="0.549019608 0.450980392 0.235294118 1" />
+      </material>
     </visual>
   </link>
@@ -26,33 +29,26 @@
     <parent link="ee_link"/>
     <child link="gripper_link"/>
-    <origin xyz="0.0 0.0 0.0" rpy="${pi} -${pi/2} 0.0" />
+    <origin xyz="0.0 0.0 0.0" rpy="0.0 ${pi/2} 0.0" />
  </joint>
   <!-- GRIPPER -->
-  <xacro:schunk_pg70 name="pg70" parent="gripper_link">
-    <origin xyz="0 0.0 0.01" rpy="0 0 0" /> <!--slightly above gazebo plane-->
-  </xacro:schunk_pg70>
-  <link name="gripper_power_box">
-    <visual>
-      <geometry>
-        <box size="0.047 0.068 0.07"/>
-      </geometry>
-    </visual>
-  </link>
-  <joint name="gripper_power_joint" type="fixed">
-    <parent link="pg70_base_link"/>
-    <child link="gripper_power_box"/>
-    <origin xyz="0.004 -0.08 0.029" rpy="0.0 0.0 ${pi/2}" />
+  <joint name="tool_joint" type="fixed">
+    <parent link="gripper_link"/>
+    <child link="tool_link"/>
+    <origin xyz="0.0 0.0 0.0" rpy="${pi} -${pi/2} 0.0" />
  </joint>
  <link name="gripper_power_cable">
     <visual>
       <geometry>
-        <cylinder length="0.025" radius="0.0075"/>
+        <cylinder length="0.03" radius="0.0075"/>
       </geometry>
+      <material name="o">
+      	 <color rgba="0.549019608 0.450980392 0.235294118 1" />
+      </material>
     </visual>
-  </link>
-  <joint name="gripper_power_cable_joint" type="fixed">
-    <parent link="gripper_power_box"/>
+ </link>
+ <joint name="gripper_power_cable_joint" type="fixed">
+    <parent link="tool_link"/>
     <child link="gripper_power_cable"/>
-    <origin xyz="0.0 0.0 -0.05" rpy="0.0 0.0 0.0" />
+    <origin xyz="0.0 -0.082 0.0" rpy="0.0 ${pi/2} 0.0" />
  </joint>
 </robot>

File: ur_description/urdf/ur3_pg70_table.urdf.xacro (robot description, xacro)
@@ -7,5 +7,5 @@
   <xacro:include filename="$(find ur_description)/urdf/ur3.urdf.xacro" />
   <!-- schunk pg70 -->
-  <xacro:include filename="$(find schunk_pg70)/urdf/pg70.urdf.xacro" />
+  <xacro:include filename="$(find schunkPG70_description)/robots/schunkPG70_description.URDF" />
   <!-- arm -->
   <xacro:ur3_robot prefix="" joint_limited="false"/>
@@ -17,4 +17,7 @@
         <box size="1.0 1.0 0.86"/>
       </geometry>
+      <material name="w">
+         <color rgba="1.0 1.0 1.0 1" />
+      </material>
     </visual>
   </link>
@@ -36,4 +39,7 @@
         <box size="0.08 0.113 0.005"/>
       </geometry>
+      <material name="o">
+         <color rgba="0.549019608 0.450980392 0.235294118 1" />
+      </material>
     </visual>
   </link>
@@ -41,33 +47,26 @@
     <parent link="ee_link"/>
     <child link="gripper_link"/>
-    <origin xyz="0.0 0.0 0.0" rpy="${pi} -${pi/2} 0.0" />
+    <origin xyz="0.0 0.0 0.0" rpy="0.0 ${pi/2} 0.0" />
  </joint>
   <!-- GRIPPER -->
-  <xacro:schunk_pg70 name="pg70" parent="gripper_link">
-    <origin xyz="0 0.0 0.01" rpy="0 0 0" /> <!--slightly above gazebo plane-->
-  </xacro:schunk_pg70>
-  <link name="gripper_power_box">
-    <visual>
-      <geometry>
-        <box size="0.047 0.068 0.07"/>
-      </geometry>
-    </visual>
-  </link>
-  <joint name="gripper_power_joint" type="fixed">
-    <parent link="pg70_base_link"/>
-    <child link="gripper_power_box"/>
-    <origin xyz="0.004 -0.08 0.029" rpy="0.0 0.0 ${pi/2}" />
+  <joint name="tool_joint" type="fixed">
+    <parent link="gripper_link"/>
+    <child link="tool_link"/>
+    <origin xyz="0.0 0.0 0.0" rpy="${pi} -${pi/2} 0.0" />
  </joint>
  <link name="gripper_power_cable">
     <visual>
       <geometry>
-        <cylinder length="0.025" radius="0.0075"/>
+        <cylinder length="0.03" radius="0.0075"/>
       </geometry>
+      <material name="o">
+         <color rgba="0.549019608 0.450980392 0.235294118 1" />
+      </material>
     </visual>
-  </link>
-  <joint name="gripper_power_cable_joint" type="fixed">
-    <parent link="gripper_power_box"/>
+ </link>
+ <joint name="gripper_power_cable_joint" type="fixed">
+    <parent link="tool_link"/>
     <child link="gripper_power_cable"/>
-    <origin xyz="0.0 0.0 -0.05" rpy="0.0 0.0 0.0" />
+    <origin xyz="0.0 -0.082 0.0" rpy="0.0 ${pi/2} 0.0" />
  </joint>
 </robot>

Commit message: ur3_pg70_mix

File: ur_description/urdf/ur3_pg70.urdf.xacro (robot description, xacro)
@@ -1,10 +1,9 @@
 <?xml version="1.0"?>
 <robot xmlns:xacro="http://ros.org/wiki/xacro"
-       name="ur3_pg70" >
+       name="ur3" >
   <!-- common stuff -->
   <xacro:include filename="$(find ur_description)/urdf/common.gazebo.xacro" />
   <!-- ur3 -->
   <xacro:include filename="$(find ur_description)/urdf/ur3.urdf.xacro" />
-  <!-- schunk pg70 -->
   <xacro:include filename="$(find schunkPG70_description)/robots/schunkPG70_description.URDF" />
   <!-- arm -->
@@ -25,4 +24,8 @@
       </material>
     </visual>
+    <inertial>
+      <mass value="0.2"/>
+      <inertia ixx ="0.001" ixy="0.0" ixz="0.0" iyy="0.001" iyz="0.0" izz="0.001"/>
+    </inertial>
   </link>
   <joint name="gripper_joint" type="fixed">

Commit message: setting up mano

File: ur_description/urdf/ur3_pg70.urdf.xacro (robot description, xacro)
@@ -1,18 +1,39 @@
 <?xml version="1.0"?>
 <robot xmlns:xacro="http://ros.org/wiki/xacro"
-       name="ur3" >
-  <!-- common stuff -->
-  <xacro:include filename="$(find ur_description)/urdf/common.gazebo.xacro" />
+       name="ur3_pg70" >
   <!-- ur3 -->
   <xacro:include filename="$(find ur_description)/urdf/ur3.urdf.xacro" />
-  <xacro:include filename="$(find schunkPG70_description)/robots/schunkPG70_description.URDF" />
+  <!-- schunk pg70 -->
+  <xacro:include filename="$(find schunk_pg70)/urdf/pg70.urdf.xacro" />
   <!-- arm -->
   <xacro:ur3_robot prefix="" joint_limited="false"/>
   <link name="world" />
+  <link name="box_link">
+    <visual>
+      <geometry>
+        <box size="1.0 1.0 0.86"/>
+      </geometry>
+    </visual>
+    <inertial>
+        <origin xyz="0 0 0" rpy="0 0 0"/>
+        <mass value="100"/>
+        <inertia ixx="1.0" ixy="0" ixz="0" iyy="1.0" iyz="0" izz="1.0" />
+    </inertial>
+    <collision>
+      <geometry>
+        <box size="1.0 1.0 0.86"/>
+      </geometry>
+    </collision>
+  </link>
   <joint name="world_joint" type="fixed">
     <parent link="world" />
-    <child link = "base_link" />
-    <origin xyz="0.0 0.0 0.0" rpy="0.0 0.0 0.0" />
+    <child link = "box_link" />
+    <origin xyz="0.0 0.0 0.43" rpy="0.0 0.0 0.0" />
   </joint>
+   <joint name="box_joint" type="fixed">
+    <parent link="box_link"/>
+    <child link="base_link"/>
+    <origin xyz="0.0 0.0 0.43" rpy="0 0 1.57" />
+ </joint>
  <link name="gripper_link">
     <visual>
@@ -21,24 +42,28 @@
       </geometry>
       <material name="o">
-      	 <color rgba="0.549019608 0.450980392 0.235294118 1" />
+        <color rgba="0.549019608 0.450980392 0.235294118 1" />
       </material>
     </visual>
     <inertial>
-      <mass value="0.2"/>
-      <inertia ixx ="0.001" ixy="0.0" ixz="0.0" iyy="0.001" iyz="0.0" izz="0.001"/>
+        <origin xyz="0 0 0" rpy="0 0 0"/>
+        <mass value="0.01"/>
+        <inertia ixx="0.0001" ixy="0" ixz="0" iyy="0.0001" iyz="0" izz="0.0001" />
     </inertial>
+    <collision>
+      <geometry>
+        <box size="0.08 0.113 0.005"/>
+      </geometry>
+    </collision>
   </link>
   <joint name="gripper_joint" type="fixed">
     <parent link="ee_link"/>
     <child link="gripper_link"/>
-    <origin xyz="0.0 0.0 0.0" rpy="0.0 ${pi/2} 0.0" />
+    <origin xyz="0.0 0.0 0.0" rpy="${pi} -${pi/2} 0.0" />
  </joint>
   <!-- GRIPPER -->
-  <joint name="tool_joint" type="fixed">
-    <parent link="gripper_link"/>
-    <child link="tool_link"/>
-    <origin xyz="0.0 0.0 0.0" rpy="${pi} -${pi/2} 0.0" />
- </joint>
- <link name="gripper_power_cable">
+  <xacro:schunk_pg70 name="pg70" parent="gripper_link">
+    <origin xyz="0 0.0 0.0" rpy="0 -${pi/2} 0" /> <!--slightly above gazebo plane-->
+  </xacro:schunk_pg70>
+  <link name="gripper_power_cable">
     <visual>
       <geometry>
@@ -46,12 +71,62 @@
       </geometry>
       <material name="o">
-      	 <color rgba="0.549019608 0.450980392 0.235294118 1" />
+         <color rgba="0.549019608 0.450980392 0.235294118 1" />
       </material>
     </visual>
+    <inertial>
+        <origin xyz="0 0 0" rpy="0 0 0"/>
+        <mass value="0.01"/>
+        <inertia ixx="0.0001" ixy="0" ixz="0" iyy="0.0001" iyz="0" izz="0.0001" />
+    </inertial>
+    <collision>
+      <geometry>
+        <cylinder length="0.03" radius="0.0075"/>
+      </geometry>
+    </collision>
  </link>
  <joint name="gripper_power_cable_joint" type="fixed">
-    <parent link="tool_link"/>
+    <parent link="pg70_base_link"/>
     <child link="gripper_power_cable"/>
     <origin xyz="0.0 -0.082 0.0" rpy="0.0 ${pi/2} 0.0" />
  </joint>
+  <!--<link name="gripper_power_box">
+    <visual>
+      <geometry>
+        <box size="0.047 0.068 0.07"/>
+         <material
+        name="">
+        <color
+          rgba="0.549019608 0.450980392 0.235294118 1" />
+      </material>
+      </geometry>
+    </visual>
+  </link>
+  <joint name="gripper_power_joint" type="fixed">
+    <parent link="pg70_base_link"/>
+    <child link="gripper_power_box"/>
+    <origin xyz="0.004 -0.08 0.029" rpy="0.0 0.0 ${pi/2}" />
+ </joint>
+ <link name="gripper_power_cable">
+    <visual>
+      <geometry>
+        <cylinder length="0.025" radius="0.0075"/>
+         <material
+        name="">
+        <color
+          rgba="0.549019608 0.450980392 0.235294118 1" />
+      </material>
+      </geometry>
+    </visual>
+  </link>
+  <joint name="gripper_power_cable_joint" type="fixed">
+    <parent link="gripper_power_box"/>
+    <child link="gripper_power_cable"/>
+    <origin xyz="0.0 0.0 -0.05" rpy="0.0 0.0 0.0" />
+ </joint>-->
+  <gazebo>
+      <plugin name="gazebo_ros_control" filename="libgazebo_ros_control.so">
+        <!--<robotNamespace>ur3_pg70</robotNamespace>-->
+         <robotSimType>gazebo_ros_control/DefaultRobotHWSim</robotSimType>
+      </plugin>
+  </gazebo>
 </robot>

File: ur_description/urdf/ur3_pg70_old.urdf.xacro (robot description, xacro)
@@ -1,39 +1,18 @@
 <?xml version="1.0"?>
 <robot xmlns:xacro="http://ros.org/wiki/xacro"
-       name="ur3_pg70" >
+       name="ur3" >
+  <!-- common stuff -->
+  <xacro:include filename="$(find ur_description)/urdf/common.gazebo.xacro" />
   <!-- ur3 -->
   <xacro:include filename="$(find ur_description)/urdf/ur3.urdf.xacro" />
-  <!-- schunk pg70 -->
-  <xacro:include filename="$(find schunk_pg70)/urdf/pg70.urdf.xacro" />
+  <xacro:include filename="$(find schunkPG70_description)/robots/schunkPG70_description.URDF" />
   <!-- arm -->
   <xacro:ur3_robot prefix="" joint_limited="false"/>
   <link name="world" />
-  <link name="box_link">
-    <visual>
-      <geometry>
-        <box size="1.0 1.0 0.86"/>
-      </geometry>
-    </visual>
-    <inertial>
-        <origin xyz="0 0 0" rpy="0 0 0"/>
-        <mass value="100"/>
-        <inertia ixx="1.0" ixy="0" ixz="0" iyy="1.0" iyz="0" izz="1.0" />
-    </inertial>
-    <collision>
-      <geometry>
-        <box size="1.0 1.0 0.86"/>
-      </geometry>
-    </collision>
-  </link>
   <joint name="world_joint" type="fixed">
     <parent link="world" />
-    <child link = "box_link" />
-    <origin xyz="0.0 0.0 0.43" rpy="0.0 0.0 0.0" />
+    <child link = "base_link" />
+    <origin xyz="0.0 0.0 0.0" rpy="0.0 0.0 0.0" />
   </joint>
-   <joint name="box_joint" type="fixed">
-    <parent link="box_link"/>
-    <child link="base_link"/>
-    <origin xyz="0.0 0.0 0.43" rpy="0 0 1.57" />
- </joint>
  <link name="gripper_link">
     <visual>
@@ -42,28 +21,24 @@
       </geometry>
       <material name="o">
-        <color rgba="0.549019608 0.450980392 0.235294118 1" />
+      	 <color rgba="0.549019608 0.450980392 0.235294118 1" />
       </material>
     </visual>
     <inertial>
-        <origin xyz="0 0 0" rpy="0 0 0"/>
-        <mass value="0.01"/>
-        <inertia ixx="0.0001" ixy="0" ixz="0" iyy="0.0001" iyz="0" izz="0.0001" />
+      <mass value="0.2"/>
+      <inertia ixx ="0.001" ixy="0.0" ixz="0.0" iyy="0.001" iyz="0.0" izz="0.001"/>
     </inertial>
-    <collision>
-      <geometry>
-        <box size="0.08 0.113 0.005"/>
-      </geometry>
-    </collision>
   </link>
   <joint name="gripper_joint" type="fixed">
     <parent link="ee_link"/>
     <child link="gripper_link"/>
+    <origin xyz="0.0 0.0 0.0" rpy="0.0 ${pi/2} 0.0" />
+ </joint>
+  <!-- GRIPPER -->
+  <joint name="tool_joint" type="fixed">
+    <parent link="gripper_link"/>
+    <child link="tool_link"/>
     <origin xyz="0.0 0.0 0.0" rpy="${pi} -${pi/2} 0.0" />
  </joint>
-  <!-- GRIPPER -->
-  <xacro:schunk_pg70 name="pg70" parent="gripper_link">
-    <origin xyz="0 0.0 0.0" rpy="0 -${pi/2} 0" /> <!--slightly above gazebo plane-->
-  </xacro:schunk_pg70>
-  <link name="gripper_power_cable">
+ <link name="gripper_power_cable">
     <visual>
       <geometry>
@@ -71,62 +46,12 @@
       </geometry>
       <material name="o">
-         <color rgba="0.549019608 0.450980392 0.235294118 1" />
+      	 <color rgba="0.549019608 0.450980392 0.235294118 1" />
       </material>
     </visual>
-    <inertial>
-        <origin xyz="0 0 0" rpy="0 0 0"/>
-        <mass value="0.01"/>
-        <inertia ixx="0.0001" ixy="0" ixz="0" iyy="0.0001" iyz="0" izz="0.0001" />
-    </inertial>
-    <collision>
-      <geometry>
-        <cylinder length="0.03" radius="0.0075"/>
-      </geometry>
-    </collision>
  </link>
  <joint name="gripper_power_cable_joint" type="fixed">
-    <parent link="pg70_base_link"/>
+    <parent link="tool_link"/>
     <child link="gripper_power_cable"/>
     <origin xyz="0.0 -0.082 0.0" rpy="0.0 ${pi/2} 0.0" />
  </joint>
-  <!--<link name="gripper_power_box">
-    <visual>
-      <geometry>
-        <box size="0.047 0.068 0.07"/>
-         <material
-        name="">
-        <color
-          rgba="0.549019608 0.450980392 0.235294118 1" />
-      </material>
-      </geometry>
-    </visual>
-  </link>
-  <joint name="gripper_power_joint" type="fixed">
-    <parent link="pg70_base_link"/>
-    <child link="gripper_power_box"/>
-    <origin xyz="0.004 -0.08 0.029" rpy="0.0 0.0 ${pi/2}" />
- </joint>
- <link name="gripper_power_cable">
-    <visual>
-      <geometry>
-        <cylinder length="0.025" radius="0.0075"/>
-         <material
-        name="">
-        <color
-          rgba="0.549019608 0.450980392 0.235294118 1" />
-      </material>
-      </geometry>
-    </visual>
-  </link>
-  <joint name="gripper_power_cable_joint" type="fixed">
-    <parent link="gripper_power_box"/>
-    <child link="gripper_power_cable"/>
-    <origin xyz="0.0 0.0 -0.05" rpy="0.0 0.0 0.0" />
- </joint>-->
-  <gazebo>
-      <plugin name="gazebo_ros_control" filename="libgazebo_ros_control.so">
-        <!--<robotNamespace>ur3_pg70</robotNamespace>-->
-         <robotSimType>gazebo_ros_control/DefaultRobotHWSim</robotSimType>
-      </plugin>
-  </gazebo>
 </robot>

Commit message: new ur3_pg70_table_moveit package

File: ur_description/urdf/ur3_pg70.urdf.xacro (robot description, xacro)
@@ -1,12 +1,11 @@
 <?xml version="1.0"?>
-<robot xmlns:xacro="http://ros.org/wiki/xacro"
-       name="ur3_pg70" >
-  <!-- ur3 -->
+<robot xmlns:xacro="http://www.ros.org/wiki/xacro"
+  name="ur3_pg70">
+<!-- schunk_pg70 -->
+  <xacro:include filename="$(find schunk_pg70)/urdf/pg70.urdf.xacro"/>
+<!-- ur3 -->
   <xacro:include filename="$(find ur_description)/urdf/ur3.urdf.xacro" />
-  <!-- schunk pg70 -->
-  <xacro:include filename="$(find schunk_pg70)/urdf/pg70.urdf.xacro" />
-  <!-- arm -->
   <xacro:ur3_robot prefix="" joint_limited="false"/>
-  <link name="world" />
+   <link name="world" />
   <link name="box_link">
     <visual>
@@ -36,5 +35,5 @@
     <origin xyz="0.0 0.0 0.43" rpy="0 0 1.57" />
  </joint>
- <link name="gripper_link">
+  <link name="gripper_link">
     <visual>
       <geometry>
@@ -47,5 +46,5 @@
     <inertial>
         <origin xyz="0 0 0" rpy="0 0 0"/>
-        <mass value="0.01"/>
+        <mass value="0.001"/>
         <inertia ixx="0.0001" ixy="0" ixz="0" iyy="0.0001" iyz="0" izz="0.0001" />
     </inertial>
@@ -62,8 +61,8 @@
  </joint>
   <!-- GRIPPER -->
-  <xacro:schunk_pg70 name="pg70" parent="gripper_link">
-    <origin xyz="0 0.0 0.0" rpy="0 -${pi/2} 0" /> <!--slightly above gazebo plane-->
+  <xacro:schunk_pg70 name="schunk_pg70" parent="gripper_link">
+    <origin xyz="0 0.0 0.0091" rpy="0 0 0" /> <!--slightly above gazebo plane-->
   </xacro:schunk_pg70>
-  <link name="gripper_power_cable">
+ <link name="gripper_power_cable">
     <visual>
       <geometry>
@@ -86,9 +85,9 @@
  </link>
  <joint name="gripper_power_cable_joint" type="fixed">
-    <parent link="pg70_base_link"/>
+    <parent link="schunk_pg70_base_link"/>
     <child link="gripper_power_cable"/>
-    <origin xyz="0.0 -0.082 0.0" rpy="0.0 ${pi/2} 0.0" />
+    <origin xyz="-0.035 -0.082 0.02" rpy="0.0 ${pi/2} 0.0" />
  </joint>
-  <!--<link name="gripper_power_box">
+  <link name="gripper_power_box">
     <visual>
       <geometry>
@@ -103,9 +102,9 @@
   </link>
   <joint name="gripper_power_joint" type="fixed">
-    <parent link="pg70_base_link"/>
+    <parent link="schunk_pg70_base_link"/>
     <child link="gripper_power_box"/>
-    <origin xyz="0.004 -0.08 0.029" rpy="0.0 0.0 ${pi/2}" />
+    <origin xyz="0.004 -0.08 0.03" rpy="0.0 0.0 ${pi/2}" />
  </joint>
- <link name="gripper_power_cable">
+ <!--<link name="gripper_power_cable">
     <visual>
       <geometry>

File: ur_description/urdf/ur3_table.urdf.xacro (robot description, xacro)
@@ -29,3 +29,7 @@
     <origin xyz="0.0 0.0 0.43" rpy="0 0 1.57" />
  </joint>
+<!--astra  -->
+ <xacro:include filename="$(find ur_description)/urdf/sensors/kinect.urdf.xacro"/>
+<!--attach the kinect to the robot -->
+ <xacro:sensor_kinect  parent="base_link"/>
 </robot>

Commit message: Real ur3_pg70 controller

File: ur_description/urdf/ur3_pg70.urdf.xacro (robot description, xacro)
@@ -106,21 +106,11 @@
     <origin xyz="0.004 -0.08 0.03" rpy="0.0 0.0 ${pi/2}" />
  </joint>
- <!--<link name="gripper_power_cable">
-    <visual>
-      <geometry>
-        <cylinder length="0.025" radius="0.0075"/>
-         <material
-        name="">
-        <color
-          rgba="0.549019608 0.450980392 0.235294118 1" />
-      </material>
-      </geometry>
-    </visual>
+ <joint name="ar_marker_joint" type="fixed">
+    <parent link="base_link"/>
+    <child link="ar_marker_link"/>
+    <origin xyz="-0.392 0.412 0.00" rpy="0.0 0.0 0.0" />
+ </joint>
+ <link name="ar_marker_link">
   </link>
-  <joint name="gripper_power_cable_joint" type="fixed">
-    <parent link="gripper_power_box"/>
-    <child link="gripper_power_cable"/>
-    <origin xyz="0.0 0.0 -0.05" rpy="0.0 0.0 0.0" />
- </joint>-->
   <gazebo>
       <plugin name="gazebo_ros_control" filename="libgazebo_ros_control.so">

Commit message: grasping

File: ur_description/urdf/ur3_pg70.urdf.xacro (robot description, xacro)
@@ -67,5 +67,5 @@
     <visual>
       <geometry>
-        <cylinder length="0.03" radius="0.0075"/>
+        <cylinder length="0.035" radius="0.012"/>
       </geometry>
       <material name="o">
@@ -80,17 +80,17 @@
     <collision>
       <geometry>
-        <cylinder length="0.03" radius="0.0075"/>
+        <cylinder length="0.035" radius="0.012"/>
       </geometry>
     </collision>
  </link>
  <joint name="gripper_power_cable_joint" type="fixed">
-    <parent link="schunk_pg70_base_link"/>
+    <parent link="gripper_power_box"/>
     <child link="gripper_power_cable"/>
-    <origin xyz="-0.035 -0.082 0.02" rpy="0.0 ${pi/2} 0.0" />
+    <origin xyz="-0.01 -0.042 -0.011" rpy="${pi/2} 0.0 0.0" />
  </joint>
   <link name="gripper_power_box">
     <visual>
       <geometry>
-        <box size="0.047 0.068 0.07"/>
+        <box size="0.047 0.072 0.072"/>
          <material
         name="">
@@ -109,5 +109,5 @@
     <parent link="base_link"/>
     <child link="ar_marker_link"/>
-    <origin xyz="-0.392 0.412 0.00" rpy="0.0 0.0 0.0" />
+    <origin xyz="-0.41 0.41 0.00" rpy="0.0 0.0 0.0" />
  </joint>
  <link name="ar_marker_link">

Commit message: demo construct

File: ur_description/urdf/ur3_pg70.urdf.xacro (robot description, xacro)
@@ -100,4 +100,9 @@
       </geometry>
     </visual>
+    <collision>
+      <geometry>
+       <box size="0.047 0.072 0.072"/>
+      </geometry>
+    </collision>
   </link>
   <joint name="gripper_power_joint" type="fixed">
